File: hardware/esp-rust-board/esp-rust-board.kicad_pcb (KiCad board)
At the start: 2 copper layers, 22.9 x 63.5 mm, 82 parts, among them J1 USB4105-GF-A, J2 MOTOR L, J3 MOTOR R, J5 LED L, J6 LED R, Q1 DMG3415U, Q2 Si2319CDS, Q3 Si2319CDS, Q4 MMBT3904, Q5 MMBT3904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

Commit message: Place components on PCB
Parts:
- removed J5: LED L, Connector_JST:JST_PH_B2B-PH-SM4-TB_1x02-1MP_P2.00mm_Vertical
- removed J6: LED R, Connector_JST:JST_PH_B2B-PH-SM4-TB_1x02-1MP_P2.00mm_Vertical
- removed Q4, Q5: MMBT3904, Package_TO_SOT_SMD:SOT-23
- removed R22, R24: 470R 1%, Resistor_SMD:R_0402_1005Metric
- removed R23, R25: 10kR 1%, Resistor_SMD:R_0402_1005Metric
- removed TP2: IMU_INT2, TestPoint:TestPoint_Pad_D1.0mm
- added H1: MountingHole_Pad, TestPoint:TestPoint_Keystone_5005-5009_Compact, F.Cu at (157.0, 126.0)
- added H2: MountingHole_Pad, TestPoint:TestPoint_Keystone_5005-5009_Compact, F.Cu at (139.2, 126.0)
- added J7: SERVO R, Connector_PinSocket_2.00mm:PinSocket_1x03_P2.00mm_Vertical, F.Cu at (138.5, 93.8)
- added J8: SERVO R, Connector_PinSocket_2.00mm:PinSocket_1x03_P2.00mm_Vertical, F.Cu at (157.8, 93.8)
- J2, J3: footprint Connector_JST:JST_PH_B2B-PH-SM4-TB_1x02-1MP_P2.00mm_Vertical -> Connector_PinHeader_2.00mm:PinHeader_1x02_P2.00mm_Vertical
- moved J3 98.0 mm to (157.8, 99.0), turned to 180 degrees
- moved D11 93.6 mm to (155.0, 97.9), turned to 90 degrees
- moved C3 88.8 mm to (153.2, 98.0), turned to -90 degrees
- moved R21 86.8 mm to (148.6, 98.2), turned to -90 degrees
- moved R20 86.8 mm to (148.6, 96.2), turned to -90 degrees
- moved Q3 85.0 mm to (151.0, 97.0), turned to -90 degrees
- moved R16 69.6 mm to (147.5, 98.2), turned to -90 degrees
- moved R13 69.5 mm to (147.5, 96.2), turned to -90 degrees
- moved J2 67.1 mm to (138.5, 99.0), turned to 180 degrees
- moved C1 65.4 mm to (143.0, 98.0), turned to -90 degrees
- moved D10 64.1 mm to (141.2, 97.8), turned to 90 degrees
- moved Q2 62.0 mm to (145.2, 97.1), turned to -90 degrees
- moved U9 44.4 mm to (150.8, 92.5)
- moved C21 44.3 mm to (153.0, 92.8), turned to -90 degrees
- moved C20 42.1 mm to (152.8, 89.0), turned to 90 degrees
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Connections:
- R11 pad 1: IO2 -> IO7
- R13 pad 1: IO7 -> IO4
- R20 pad 1: IO6 -> IO5
- TP1 pad 1: IO20_RX -> IO21_TX
- TP3 pad 1: IO21_TX -> IO20_RX
- U2 pad 9: Net-(U2-INT2) -> unconnected-(U2-INT2-Pad9)
- U3 pad 13: IO1 -> unconnected-(U3-GPIO1/ADC1_CH1/XTAL_32K_N-Pad13)
- U3 pad 5: IO2 -> unconnected-(U3-GPIO2/ADC1_CH2-Pad5)
- U3 pad 6: IO3 -> unconnected-(U3-GPIO3/ADC1_CH3-Pad6)
Routing:
- net IO2: track 38.2 -> 0.00 mm, vias 2 -> 0
- net +BATT: track 35.5 -> 71.4 mm, vias 2 -> 1
- net IO3: track 31.1 -> 0.00 mm, vias 1 -> 0
- net IO1: track 25.1 -> 0.00 mm, vias 1 -> 0
- net IO20_RX: track 43.9 -> 22.6 mm, vias 5 -> 4
- net IO21_TX: track 43.8 -> 22.8 mm, vias 5 -> 4
- net IO8_SCL: track 42.9 -> 27.1 mm
- net IO7: track 26.2 -> 13.1 mm, vias 1 -> 2
- net IO4: track 25.5 -> 17.3 mm, vias 1 -> 2
- net Net-(D10-A): track 0.00 -> 7.78 mm
- net Net-(D11-A): track 0.00 -> 7.76 mm
- net IO5: track 25.6 -> 18.3 mm, vias 1 -> 2
- net IO0: track 25.2 -> 18.1 mm, vias 1 -> 0
- net CHIP_PU: track 49.9 -> 43.4 mm
- net Net-(U9-CAP): track 0.00 -> 5.88 mm, vias 0 -> 2
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
Commit message: Minor corrections
Parts:
- removed D2: LED, LED_SMD:LED_0603_1608Metric
- removed R10: 470R 1%, Resistor_SMD:R_0402_1005Metric
- moved R13 0.10 mm to (147.6, 96.2)
- moved R16 0.10 mm to (147.6, 98.2)
- moved C1 0.05 mm to (142.9, 98.0)
- moved R20 0.05 mm to (148.7, 96.2)
- moved R21 0.05 mm to (148.7, 98.2)
Routing:
- net +3V3: track 53.3 -> 62.2 mm, vias 13 -> 12
- net +BATT: track 71.4 -> 70.2 mm
- net Net-(U8-CSB): track 3.03 -> 2.45 mm
- net GND: vias 155 -> 157

Commit message: Design completed
Parts:
- added D2: LED, LED_SMD:LED_0603_1608Metric, F.Cu at (157.0, 79.3)
- added J4: LED L, Connector_PinHeader_2.00mm:PinHeader_1x02_P2.00mm_Vertical, F.Cu at (138.5, 86.5)
- added Q4: MMBT3904, Package_TO_SOT_SMD:SOT-23, F.Cu at (142.8, 86.0)
- added R10: 470R 1%, Resistor_SMD:R_0402_1005Metric, F.Cu at (157.0, 82.0)
- added R22: 470R 1%, Resistor_SMD:R_0402_1005Metric, F.Cu at (143.8, 83.7)
- added R23: 10kR 1%, Resistor_SMD:R_0402_1005Metric, F.Cu at (141.8, 88.3)
- C1, C3: value 1uF -> 1uF 16V
- moved TP3 0.90 mm to (138.0, 79.5)
- moved TP1 0.75 mm to (138.0, 77.5)
- moved C19 0.20 mm to (148.0, 92.5)
- moved C21 0.20 mm to (153.2, 92.8)
Connections:
- J7 pad 1: IO0 -> IO1
- U3 pad 13: unconnected-(U3-GPIO1/ADC1_CH1/XTAL_32K_N-Pad13) -> IO1
Routing:
- net IO1: track 0.00 -> 17.8 mm
- net IO0: track 18.1 -> 2.47 mm
- net Net-(Q4-B): track 0.00 -> 7.94 mm
- net +BATT: track 70.2 -> 76.5 mm
- net Net-(J4-Pin_2): track 0.00 -> 3.98 mm
- net CHIP_PU: track 43.4 -> 45.5 mm
- net Net-(D2-A): track 0.00 -> 1.42 mm
- net IO21_TX: track 22.8 -> 21.7 mm
- net +3V3: track 62.2 -> 61.2 mm, vias 12 -> 16
- net IO9_BOOT: track 56.3 -> 56.9 mm, vias 4 -> 2
- net IO20_RX: track 22.6 -> 22.1 mm
- net GND: vias 157 -> 195
Other:
- board text added: "REV 1"
- board text added: "RX"
- board text added: "TX"
